Commit message: fix an important bug

File: urdf/robot.urdf (robot description, URDF)
Before this commit: robot HLRobot, 8 links, 7 joints
Links:
- link base_link: geometry collision mesh filename=package://hlrobot/meshes/base_link.STL; visual mesh filename=package://hlrobot/meshes/base_link.STL
- link link1: geometry collision mesh filename=package://hlrobot/meshes/link1.STL; visual mesh filename=package://hlrobot/meshes/link1.STL
- link link2: geometry collision mesh filename=package://hlrobot/meshes/link2.STL; visual mesh filename=package://hlrobot/meshes/link2.STL
- link link3: geometry collision mesh filename=package://hlrobot/meshes/link3.STL; visual mesh filename=package://hlrobot/meshes/link3.STL
- link link4: geometry collision mesh filename=package://hlrobot/meshes/link4.STL; visual mesh filename=package://hlrobot/meshes/link4.STL
- link link5: geometry collision mesh filename=package://hlrobot/meshes/link5.STL; visual mesh filename=package://hlrobot/meshes/link5.STL
- link link6: geometry collision mesh filename=package://hlrobot/meshes/link6.STL; visual mesh filename=package://hlrobot/meshes/link6.STL
