Commit message: finish robot model and function 1

File: urdf/arm.xacro (robot description, xacro)
@@ -1,4 +1,4 @@
 <?xml version="1.0" encoding="utf-8"?>
-<robot xmlns:xacro="http://ros.org/wiki/xacro" name="HLRobot">
+<robot xmlns:xacro="http://ros.org/wiki/xacro" name="arm">
     <link name="base_footprint">
         <visual>
@@ -274,3 +274,44 @@
         <plugin name="gazebo_ros_control" filename="libgazebo_ros_control.so"/>
     </gazebo>
+    <!-- Tools -->
+    <link name="tool1">
+        <visual>
+            <origin xyz="0 0 0" rpy="0 0 0" />
+            <geometry>
+                <cylinder radius="0.005" length ="0.2"/>
+            </geometry>
+        </visual>
+        <collision>
+            <origin xyz="0 0 0" rpy="0 0 0" />
+            <geometry>
+                <sphere radius="0.001"/>
+            </geometry>
+        </collision>
+    </link>
+    <joint name="link62tool1" type="fixed">
+        <origin xyz="-0.1 0 -0.005" rpy="1.50707 0 1.50707" />
+        <parent link="link6" />
+        <child link="tool1" />
+        <axis xyz="0 0 0" />
+    </joint>
+    <link name="tool2">
+        <visual>
+            <origin xyz="0 0 0" rpy="0 0 0" />
+            <geometry>
+                <sphere radius="0.02" />
+            </geometry>
+        </visual>
+        <collision>
+            <origin xyz="0 0 0" rpy="0 0 0" />
+            <geometry>
+                <sphere radius="0.02"/>
+            </geometry>
+        </collision>
+    </link>
+    <joint name="tool12tool2" type="fixed">
+        <origin xyz="0 0 -0.1" rpy="0 0 0" />
+        <parent link="tool1" />
+        <child link="tool2" />
+        <axis xyz="0 0 0" />
+    </joint>
 </robot>

Commit message: fix transform bugs

File: urdf/arm.xacro (robot description, xacro)
@@ -41,5 +41,4 @@
         <parent link="base_footprint" />
         <child link="base_link" />
-        <axis xyz="0 0 -1" />
     </joint>
     <link name="link1">
@@ -293,5 +292,4 @@
         <parent link="link6" />
         <child link="tool1" />
-        <axis xyz="0 0 0" />
     </joint>
     <link name="tool2">
@@ -313,5 +311,4 @@
         <parent link="tool1" />
         <child link="tool2" />
-        <axis xyz="0 0 0" />
     </joint>
 </robot>

Commit message: Format urdf

File: urdf/arm.xacro (robot description, xacro)
@@ -273,42 +273,3 @@
         <plugin name="gazebo_ros_control" filename="libgazebo_ros_control.so"/>
     </gazebo>
-    <!-- Tools -->
-    <link name="tool1">
-        <visual>
-            <origin xyz="0 0 0" rpy="0 0 0" />
-            <geometry>
-                <cylinder radius="0.005" length ="0.2"/>
-            </geometry>
-        </visual>
-        <collision>
-            <origin xyz="0 0 0" rpy="0 0 0" />
-            <geometry>
-                <sphere radius="0.001"/>
-            </geometry>
-        </collision>
-    </link>
-    <joint name="link62tool1" type="fixed">
-        <origin xyz="-0.1 0 -0.005" rpy="1.50707 0 1.50707" />
-        <parent link="link6" />
-        <child link="tool1" />
-    </joint>
-    <link name="tool2">
-        <visual>
-            <origin xyz="0 0 0" rpy="0 0 0" />
-            <geometry>
-                <sphere radius="0.02" />
-            </geometry>
-        </visual>
-        <collision>
-            <origin xyz="0 0 0" rpy="0 0 0" />
-            <geometry>
-                <sphere radius="0.02"/>
-            </geometry>
-        </collision>
-    </link>
-    <joint name="tool12tool2" type="fixed">
-        <origin xyz="0 0 -0.1" rpy="0 0 0" />
-        <parent link="tool1" />
-        <child link="tool2" />
-    </joint>
 </robot>

File: urdf/robot.xacro (robot description, xacro)
@@ -1,5 +1,5 @@
-<?xml version="1.0" encoding="utf-8"?>
+<?xml version="1.0"?>
 <robot xmlns:xacro="http://ros.org/wiki/xacro" name="HLRobot">
-    <xacro:include filename="/home/liuxiao/catkin_ws/src/HLRobot_gazebo/urdf/arm.xacro" />
-    <!-- <xacro:include filename="tool.xacro" /> -->
+    <xacro:include filename="arm.xacro" />
+    <xacro:include filename="tool.xacro" />
 </robot>

File: urdf/tool.xacro (robot description, xacro)
@@ -1,9 +1,10 @@
 <?xml version="1.0" encoding="utf-8"?>
 <robot xmlns:xacro="http://ros.org/wiki/xacro" name="HLRobot">
+    <!-- Tools -->
     <link name="tool1">
         <visual>
             <origin xyz="0 0 0" rpy="0 0 0" />
             <geometry>
-                <cylinder radius="0.01" length ="0.2"/>
+                <cylinder radius="0.005" length ="0.2"/>
             </geometry>
         </visual>
@@ -16,8 +17,26 @@
     </link>
     <joint name="link62tool1" type="fixed">
-        <origin xyz="0 0 0" rpy="0 0 0" />
+        <origin xyz="-0.1 0 -0.005" rpy="1.50707 0 1.50707" />
         <parent link="link6" />
         <child link="tool1" />
-        <axis xyz="0 0 0" />
+    </joint>
+    <link name="tool2">
+        <visual>
+            <origin xyz="0 0 0" rpy="0 0 0" />
+            <geometry>
+                <sphere radius="0.02" />
+            </geometry>
+        </visual>
+        <collision>
+            <origin xyz="0 0 0" rpy="0 0 0" />
+            <geometry>
+                <sphere radius="0.02"/>
+            </geometry>
+        </collision>
+    </link>
+    <joint name="tool12tool2" type="fixed">
+        <origin xyz="0 0 -0.1" rpy="0 0 0" />
+        <parent link="tool1" />
+        <child link="tool2" />
     </joint>
 </robot>

Commit message: finish play

File: urdf/arm.xacro (robot description, xacro)
@@ -38,5 +38,5 @@
     </link>
     <joint name="base_footprint2base_link" type="fixed">
-        <origin xyz="0 0 0" rpy="0 0 0" />
+        <origin xyz="-0.03 0 0" rpy="0 0 -1.5707" />
         <parent link="base_footprint" />
         <child link="base_link" />
@@ -68,5 +68,5 @@
         <parent link="base_link" />
         <child link="link1" />
-        <axis xyz="0 0 -1" />
+        <axis xyz="0 0 1" />
     </joint>
     <link name="link2">
@@ -152,5 +152,5 @@
         <parent link="link3" />
         <child link="link4" />
-        <axis xyz="0 0 -1" />
+        <axis xyz="0 0 1" />
     </joint>
     <link name="link5">

Commit message: calibration is OK

File: urdf/arm.xacro (robot description, xacro)
@@ -210,4 +210,23 @@
         <axis xyz="0 0 -1" />
     </joint>
+    <link name="tool_frame">
+        <visual>
+            <origin xyz="0 0 0" rpy="0 0 0" />
+            <geometry>
+                <sphere radius="0.001"/>
+            </geometry>
+        </visual>
+        <collision>
+            <origin xyz="0 0 0" rpy="0 0 0" />
+            <geometry>
+                <sphere radius="0.001"/>
+            </geometry>
+        </collision>
+    </link>
+    <joint name="joint62toolframe" type="fixed">
+        <origin xyz="0 0 0" rpy="3.14159 0 -1.5707" />
+        <parent link="link6" />
+        <child link="tool_frame" />
+    </joint>
     <!-- transmission -->
     <transmission name="joint1_trans">

File: urdf/tool.xacro (robot description, xacro)
@@ -17,5 +17,5 @@
     </link>
     <joint name="link62tool1" type="fixed">
-        <origin xyz="0.1 0 -0.005" rpy="1.50707 0 -1.50707" />
+        <origin xyz="-0.1 0 -0.005" rpy="-1.50707 0 -1.50707" />
         <parent link="link6" />
         <child link="tool1" />

Commit message: repair the world

File: urdf/arm.xacro (robot description, xacro)
@@ -292,3 +292,9 @@
         <plugin name="gazebo_ros_control" filename="libgazebo_ros_control.so"/>
     </gazebo>
+    <!-- gazebo -->
+    <gazebo reference="base_link">
+            <material>Gazebo/White</material>
+            <mu1>500</mu1>
+            <mu2>500</mu2>
+     </gazebo>
 </robot>

Commit message: update launch

File: urdf/arm.xacro (robot description, xacro)
@@ -18,5 +18,5 @@
         <inertial>
             <origin xyz="0.000405214557039469 0.00397651461292238 0.169839806497255" rpy="0 0 0" />
-            <mass value="500" />
+            <mass value="50" />
             <inertia ixx="0.10581489524942" ixy="0.000527121157082633" ixz="-7.56911148408879E-05" iyy="0.107337475091701" iyz="-0.00154168528325628" izz="0.101543534070196" />
         </inertial>
@@ -292,9 +292,9 @@
         <plugin name="gazebo_ros_control" filename="libgazebo_ros_control.so"/>
     </gazebo>
-    <!-- gazebo -->
-    <gazebo reference="base_link">
-        <material>Gazebo/White</material>
-        <mu1>500</mu1>
-        <mu2>500</mu2>
-    </gazebo>
+    <!-- Used for fixing robot to Gazebo 'base_link' -->
+    <link name="world"/>
+    <joint name="fixed" type="fixed">
+        <parent link="world"/>
+        <child link="base_footprint"/>
+    </joint>
 </robot>
