Commit message: regenerate model

File: urdf/robot.xacro (robot description, xacro)
@@ -1,279 +1,5 @@
 <?xml version="1.0" encoding="utf-8"?>
-<!-- This URDF was automatically created by SolidWorks to URDF Exporter! Originally created by Stephen Brawner (brawner@gmail.com)
-     Commit Version: 1.6.0-1-g15f4949  Build Version: 1.6.7594.29634
-     For more information, please see http://wiki.ros.org/sw_urdf_exporter -->
 <robot xmlns:xacro="http://ros.org/wiki/xacro" name="HLRobot">
-    <link name="base_footprint">
-        <visual>
-            <origin xyz="0 0 0" rpy="0 0 0" />
-            <geometry>
-                <sphere radius="0.001"/>
-            </geometry>
-        </visual>
-        <collision>
-            <origin xyz="0 0 0" rpy="0 0 0" />
-            <geometry>
-                <sphere radius="0.001"/>
-            </geometry>
-        </collision>
-    </link>
-    <link name="base_link">
-        <inertial>
-            <origin xyz="0.000539573047060369 -0.0205236208982336 0.327509567901413" rpy="0 0 0" />
-            <mass value="5.47150127694947" />
-            <inertia ixx="0.10581489524942" ixy="0.000527121157082598" ixz="-7.56911148408964E-05" iyy="0.107337475091701" iyz="-0.0015416852832563" izz="0.101543534070196" />
-        </inertial>
-        <visual>
-            <origin xyz="0 0 0" rpy="0 0 0" />
-            <geometry>
-                <mesh filename="package://hlrobot_gazebo/meshes/base_link.STL" />
-            </geometry>
-            <material name="">
-                <color rgba="0.52156862745098 0.541176470588235 0.541176470588235 1" />
-            </material>
-        </visual>
-        <collision>
-            <origin xyz="0 0 0" rpy="0 0 0" />
-            <geometry>
-                <mesh filename="package://hlrobot_gazebo/meshes/base_link.STL" />
-            </geometry>
-        </collision>
-    </link>
-    <joint name="base_footprint2base_link" type="fixed">
-        <origin xyz="0 0 0" rpy="0 0 0" />
-        <parent link="base_footprint" />
-        <child link="base_link" />
-        <axis xyz="0 0 -1" />
-    </joint>
-    <link name="link1">
-        <inertial>
-            <origin xyz="0.0061899 0.00043445 0.10849" rpy="0 0 0" />
-            <mass value="5.8652" />
-            <inertia ixx="0.07013" ixy="2.32E-05" ixz="0.00092902" iyy="0.046945" iyz="-0.00029004" izz="0.047319" />
-        </inertial>
-        <visual>
-            <origin xyz="0 0 0" rpy="0 0 0" />
-            <geometry>
-                <mesh filename="package://hlrobot_gazebo/meshes/link1.STL" />
-            </geometry>
-            <material name="">
-                <color rgba="1 1 1 1" />
-            </material>
-        </visual>
-        <collision>
-            <origin xyz="0 0 0" rpy="0 0 0" />
-            <geometry>
-                <mesh filename="package://hlrobot_gazebo/meshes/link1.STL" />
-            </geometry>
-        </collision>
-    </link>
-    <joint name="joint1" type="continuous">
-        <origin xyz="0 0 0.45467" rpy="0 0 1.5708" />
-        <parent link="base_link" />
-        <child link="link1" />
-        <axis xyz="0 0 -1" />
-    </joint>
-    <link name="link2">
-        <inertial>
-            <origin xyz="-0.012947 0.19509 -7.4996E-05" rpy="0 0 0" />
-            <mass value="10.107" />
-            <inertia ixx="0.26326" ixy="0.0038614" ixz="5.6195E-08" iyy="0.051701" iyz="-2.0524E-05" izz="0.24255" />
-        </inertial>
-        <visual>
-            <origin xyz="0 0 0" rpy="0 0 0" />
-            <geometry>
-                <mesh filename="package://hlrobot_gazebo/meshes/link2.STL" />
-            </geometry>
-            <material name="">
-                <color rgba="1 1 1 1" />
-            </material>
-        </visual>
-        <collision>
-            <origin xyz="0 0 0" rpy="0 0 0" />
-            <geometry>
-                <mesh filename="package://hlrobot_gazebo/meshes/link2.STL" />
-            </geometry>
-        </collision>
-    </link>
-    <joint name="joint2" type="continuous">
-        <origin xyz="0 0.0001 0.18914" rpy="1.5708 0 0"/>
-        <parent link="link1" />
-        <child link="link2" />
-        <axis xyz="0 0 -1" />
-    </joint>
-    <link name="link3">
-        <inertial>
-            <origin xyz="-0.00010884 -0.013936 -0.00014291" rpy="0 0 0" />
-            <mass value="2.6574" />
-            <inertia ixx="0.0088618" ixy="1.3764E-05" ixz="1.2847E-08" iyy="0.0067874" iyz="5.738E-06" izz="0.0093701" />
-        </inertial>
-        <visual>
-            <origin xyz="0 0 0" rpy="0 0 0" />
-            <geometry>
-                <mesh filename="package://hlrobot_gazebo/meshes/link3.STL" />
-            </geometry>
-            <material name="">
-                <color rgba="1 1 1 1" />
-            </material>
-        </visual>
-        <collision>
-            <origin xyz="0 0 0" rpy="0 0 0" />
-            <geometry>
-                <mesh filename="package://hlrobot_gazebo/meshes/link3.STL" />
-            </geometry>
-        </collision>
-    </link>
-    <joint name="joint3" type="continuous">
-        <origin xyz="0 0.45186 -0.0001" rpy="0 0 0" />
-        <parent link="link2" />
-        <child link="link3" />
-        <axis xyz="0 0 -1" />
-    </joint>
-    <link name="link4">
-        <inertial>
-            <origin xyz="-8.8639E-05 -8.2193E-05 0.18467" rpy="0 0 0" />
-            <mass value="4.3453" />
-            <inertia ixx="0.047411" ixy="4.2128E-08" ixz="-5.2664E-05" iyy="0.044812" iyz="6.5921E-05" izz="0.0095846" />
-        </inertial>
-        <visual>
-            <origin xyz="0 0 0" rpy="0 0 0" />
-            <geometry>
-                <mesh filename="package://hlrobot_gazebo/meshes/link4.STL" />
-            </geometry>
-            <material name="">
-                <color rgba="1 1 1 1" />
-            </material>
-        </visual>
-        <collision>
-            <origin xyz="0 0 0" rpy="0 0 0" />
-            <geometry>
-                <mesh filename="package://hlrobot_gazebo/meshes/link4.STL" />
-            </geometry>
-        </collision>
-    </link>
-    <joint name="joint4" type="continuous">
-        <origin xyz="0 0.08 0" rpy="-1.5708 0 0" />
-        <parent link="link3" />
-        <child link="link4" />
-        <axis xyz="0 0 -1" />
-    </joint>
-    <link name="link5">
-        <inertial>
-            <origin xyz="-9.0182E-09 0.015067 0.00097029" rpy="0 0 0" />
-            <mass value="0.48663" />
-            <inertia ixx="0.00067095" ixy="-1.0278E-10" ixz="-6.7463E-10" iyy="0.00039174" iyz="1.1694E-05" izz="0.00062744" />
-        </inertial>
-        <visual>
-            <origin xyz="0 0 0" rpy="0 0 0" />
-            <geometry>
-                <mesh filename="package://hlrobot_gazebo/meshes/link5.STL" />
-            </geometry>
-            <material name="">
-                <color rgba="1 1 1 1" />
-            </material>
-        </visual>
-        <collision>
-            <origin xyz="0 0 0" rpy="0 0 0" />
-            <geometry>
-                <mesh filename="package://hlrobot_gazebo/meshes/link5.STL" />
-            </geometry>
-        </collision>
-    </link>
-    <joint name="joint5" type="continuous">
-        <origin xyz="0 0 0.37" rpy="1.5708 0 0" />
-        <parent link="link4" />
-        <child link="link5" />
-        <axis xyz="0 0 -1" />
-    </joint>
-    <link name="link6">
-        <inertial>
-            <origin xyz="0.00018284 0.0001011 0.0031318" rpy="0 0 0" />
-            <mass value="0.0077858" />
-            <inertia ixx="9.1978E-07" ixy="-1.27E-08" ixz="-1.5206E-09" iyy="9.0815E-07" iyz="-4.1377E-10" izz="1.7718E-06" />
-        </inertial>
-        <visual>
-            <origin xyz="0 0 0" rpy="0 0 0" />
-            <geometry>
-                <mesh filename="package://hlrobot_gazebo/meshes/link6.STL" />
-            </geometry>
-            <material name="">
-                <color rgba="1 1 1 1" />
-            </material>
-        </visual>
-        <collision>
-            <origin xyz="0 0 0" rpy="0 0 0" />
-            <geometry>
-                <mesh filename="package://hlrobot_gazebo/meshes/link6.STL" />
-            </geometry>
-        </collision>
-    </link>
-    <joint name="joint6" type="continuous">
-        <origin xyz="0 0.0773 0" rpy="1.5708 1.5708 0" />
-        <parent link="link5" />
-        <child link="link6" />
-        <axis xyz="0 0 -1" />
-    </joint>
-    <!-- transmission -->
-    <transmission name="joint1_trans">
-        <type>transmission_interface/SimpleTransmission</type>
-        <joint name="joint1">
-            <hardwareInterface>hardware_interface/PositionJointInterface</hardwareInterface>
-        </joint>
-        <actuator name="motor1">
-            <mechanicalReduction>1</mechanicalReduction>
-        </actuator>
-    </transmission>
-    <!-- transmission -->
-    <transmission name="join2_trans">
-        <type>transmission_interface/SimpleTransmission</type>
-        <joint name="joint2">
-            <hardwareInterface>hardware_interface/PositionJointInterface</hardwareInterface>
-        </joint>
-        <actuator name="motor2">
-            <mechanicalReduction>1</mechanicalReduction>
-        </actuator>
-    </transmission>
-    <!-- transmission -->
-    <transmission name="joint3_trans">
-        <type>transmission_interface/SimpleTransmission</type>
-        <joint name="joint3">
-            <hardwareInterface>hardware_interface/PositionJointInterface</hardwareInterface>
-        </joint>
-        <actuator name="motor3">
-            <mechanicalReduction>1</mechanicalReduction>
-        </actuator>
-    </transmission>
-    <!-- transmission -->
-    <transmission name="joint4_trans">
-        <type>transmission_interface/SimpleTransmission</type>
-        <joint name="joint4">
-            <hardwareInterface>hardware_interface/PositionJointInterface</hardwareInterface>
-        </joint>
-        <actuator name="motor4">
-            <mechanicalReduction>1</mechanicalReduction>
-        </actuator>
-    </transmission>
-    <!-- transmission -->
-    <transmission name="joint5_trans">
-        <type>transmission_interface/SimpleTransmission</type>
-        <joint name="joint5">
-            <hardwareInterface>hardware_interface/PositionJointInterface</hardwareInterface>
-        </joint>
-        <actuator name="motor5">
-            <mechanicalReduction>1</mechanicalReduction>
-        </actuator>
-    </transmission>
-    <transmission name="joint6_trans">
-        <type>transmission_interface/SimpleTransmission</type>
-        <joint name="joint6">
-            <hardwareInterface>hardware_interface/PositionJointInterface</hardwareInterface>
-        </joint>
-        <actuator name="motor6">
-            <mechanicalReduction>1</mechanicalReduction>
-        </actuator>
-    </transmission>
-    <!-- ROS Control plugin for Gazebo -->
-    <gazebo>
-        <plugin name="gazebo_ros_control" filename="libgazebo_ros_control.so"/>
-    </gazebo>
+    <xacro:include filename="/home/liuxiao/catkin_ws/src/HLRobot_gazebo/urdf/arm.xacro" />
+    <!-- <xacro:include filename="tool.xacro" /> -->
 </robot>

Commit message: add camera for hand eye calibration

File: urdf/robot.xacro (robot description, xacro)
@@ -1,5 +1,9 @@
 <?xml version="1.0"?>
 <robot xmlns:xacro="http://ros.org/wiki/xacro" name="HLRobot">
+    <xacro:property name="PI" value="3.1415926535897931"/>
     <xacro:include filename="arm.xacro" />
-    <xacro:include filename="tool.xacro" />
+    <xacro:include filename="CameraSensor.xacro"/>
+    <xacro:Macro_CameraROS name="camera" parent="tool_frame" frame="camera_link" image_topic="image_raw" fov="1.396" hz="10" width="640" height="480">
+        <origin xyz="0 0 0.2" rpy="0 0 0" />
+    </xacro:Macro_CameraROS>
 </robot>
