Commit message: add more calibration board

File: hlrobot_gazebo/urdf/robot.xacro (robot description, xacro)
@@ -7,3 +7,9 @@
         <origin xyz="0.05 0 0.2" rpy="0 0 0" />
     </xacro:Macro_CameraROS>
+    <link name="camera_projection_frame"/>
+    <joint name="camera_joint" type="fixed">
+        <origin xyz="0 0 0" rpy="-1.5707 0 -1.5707" />
+        <parent link="camera_link" />
+        <child link="camera_projection_frame" />
+    </joint>
 </robot>
