Commit message: add camera info

File: hlrobot_gazebo/urdf/CameraSensor.xacro (robot description, xacro)
@@ -58,9 +58,9 @@
                     <frameName>${frame}</frameName>
                     <hackBaseline>0.07</hackBaseline>
-                    <distortionK1>0.0</distortionK1>
-                    <distortionK2>0.0</distortionK2>
-                    <distortionK3>0.0</distortionK3>
-                    <distortionT1>0.0</distortionT1>
-                    <distortionT2>0.0</distortionT2>
+                    <distortionK1>-0.3299099196112457</distortionK1>
+                    <distortionK2>0.125097165288712</distortionK2>
+                    <distortionK3>0</distortionK3>
+                    <distortionT1>0.001174557712517122</distortionT1>
+                    <distortionT2>-0.0006193756409617658</distortionT2>
                 </plugin>
             </sensor>

File: hlrobot_gazebo/urdf/robot.xacro (robot description, xacro)
@@ -4,6 +4,6 @@
     <xacro:include filename="arm.xacro" />
     <xacro:include filename="CameraSensor.xacro"/>
-    <xacro:Macro_CameraROS name="camera" parent="tool_frame" frame="camera_link" image_topic="image_raw" fov="1.396" hz="10" width="640" height="480">
-        <origin xyz="0 0 0.2" rpy="0 0 0" />
+    <xacro:Macro_CameraROS name="camera" parent="tool_frame" frame="camera_link" image_topic="image_raw" fov="1.396" hz="10" width="1280" height="720">
+        <origin xyz="0.05 0 0.2" rpy="0 0 0" />
     </xacro:Macro_CameraROS>
 </robot>

Commit message: add eye to hand simulation

File: hlrobot_gazebo/urdf/CameraSensor.xacro (robot description, xacro)
@@ -1,5 +1,5 @@
 <?xml version="1.0"?>
 <robot xmlns:xacro="http://www.ros.org/wiki/xacro" name="Camera">
-    <xacro:property name="camera_size" value="0.08"/>
+    <xacro:property name="camera_size" value="0.02"/>
     <xacro:macro name="Macro_CameraROS" params="name parent frame image_topic hz *origin fov width height">
         <joint name="${name}_mount_joint" type="fixed">

File: hlrobot_gazebo/urdf/arm.xacro (robot description, xacro)
@@ -38,5 +38,5 @@
     </link>
     <joint name="base_footprint2base_link" type="fixed">
-        <origin xyz="-0.03 0 0" rpy="0 0 -1.5707" />
+        <origin xyz="0 0 0" rpy="0 0 -1.5707" />
         <parent link="base_footprint" />
         <child link="base_link" />

File: hlrobot_gazebo/urdf/robot.xacro (robot description, xacro)
@@ -4,6 +4,6 @@
     <xacro:include filename="arm.xacro" />
     <xacro:include filename="CameraSensor.xacro"/>
-    <xacro:Macro_CameraROS name="camera" parent="tool_frame" frame="camera_link" image_topic="image_raw" fov="1.396" hz="10" width="1280" height="720">
-        <origin xyz="0.05 0 0.2" rpy="0 0 0" />
+    <xacro:Macro_CameraROS name="camera" parent="tool_frame" frame="camera_link" image_topic="image_raw" fov="1.396" hz="10" width="2560" height="1920">
+        <origin xyz="0.05 0 0.05" rpy="0 0 0" />
     </xacro:Macro_CameraROS>
     <link name="camera_projection_frame"/>
